File: Hardware/BAT_SWD-Adapterboard/BAT_SWD-Adapterboard.kicad_pcb (KiCad board)
At the start: 2 copper layers, 12.9 x 15 mm, 3 parts, among them J1 Conn_01x06_Pin, J2 Header_20021121-00010C4LF, J3 Conn_01x31_Pin

Commit message: Minor adjustments to SWD-Adapterboard
Routing:
- net /SWCLK: track 14.7 -> 13.0 mm
Other:
- board text added: "S. Nicora|V1-0"
- board text added: "SWD-Adapter"
- board text removed: "SWD-Adapter (C) S. Nicora V1.0"
Changed lines of the file:
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@@
 		(tags "Through hole pin header THT 2x03 2.54mm double row")
 		(property "Reference" "J1"
-			(at 1.27 -2.33 270)
+			(at 1.27 -2.33 -90)
 			(layer "F.SilkS")
 			(hide yes)
@@
 		)
 		(property "Value" "Conn_01x06_Pin"
-			(at 1.27 7.41 270)
+			(at 1.27 7.41 -90)
 			(layer "F.Fab")
 			(hide yes)
@@
 		(at 174.8 73.9)
 		(property "Reference" "J2"
-			(at 0.27 -5.035 360)
+			(at 0.27 -5.035 0)
 			(layer "F.SilkS")
 			(hide yes)
@@
 		)
 		(property "Value" "Header_20021121-00010C4LF"
-			(at 12.97 5.015 360)
+			(at 12.97 5.015 0)
 			(layer "F.Fab")
 			(hide yes)
@@
 		(layer "Edge.Cuts")
 	)
-	(gr_text "SWD-Adapter\n(C) S. Nicora\nV1.0"
-		(at 179.8 76.7 0)
+	(gr_text "SWD-Adapter"
+		(at 179.9 72.8 0)
 		(layer "B.SilkS")
 		(effects
@@
 		)
 	)
+	(gr_text "S. Nicora|V1-0"
+		(at 179.1 71.2 270)
+		(layer "F.SilkS")
+		(effects
+			(font
+				(size 1 1)
+				(thickness 0.15)
+			)
+			(justify left bottom)
+		)
+	)
 	(gr_text "GND"
 		(at 176 77.9 0)
@@
 	(segment
 		(start 178.15 75.85)
-		(end 180.411576 73.588424)
-		(width 0.2)
-		(layer "F.Cu")
-		(net 4)
-	)
-	(segment
-		(start 180.411576 72.338782)
-		(end 180.980158 71.7702)
+		(end 180.1 73.9)
 		(width 0.2)
 		(layer "F.Cu")
@@
 	)
 	(segment
-		(start 180.411576 73.588424)
-		(end 180.411576 72.338782)
-		(width 0.2)
-		(layer "F.Cu")
-		(net 4)
-	)
-	(segment
 		(start 176.1 78.7)
 		(end 177.34 77.46)
@@
 	)
 	(segment
+		(start 180.1 72.650358)
+		(end 180.980158 71.7702)
+		(width 0.2)
+		(layer "F.Cu")
+		(net 4)
+	)
+	(segment
+		(start 177.34 75.85)
+		(end 178.15 75.85)
+		(width 0.2)
+		(layer "F.Cu")
+		(net 4)
+	)
+	(segment
 		(start 180.980158 71.7702)
 		(end 181.2 71.7702)
@@
 	)
 	(segment
-		(start 177.34 75.85)
-		(end 178.15 75.85)
+		(start 180.1 73.9)
+		(end 180.1 72.650358)
 		(width 0.2)
 		(layer "F.Cu")
@@
 	)
 	(segment
-		(start 173.6 75.62)
-		(end 173.6 80.66)
+		(start 173.665 75.685)
+		(end 173.665 80.725)
 		(width 0.2)
 		(layer "F.Cu")
@@
 	)
 	(segment
-		(start 173.6 80.66)
+		(start 173.665 80.725)
 		(end 174.815 81.875)
+		(width 0.2)
+		(layer "F.Cu")
+		(net 6)
+	)
+	(segment
+		(start 173.53 75.55)
+		(end 173.665 75.685)
+		(width 0.2)
+		(layer "F.Cu")
+		(net 6)
+	)
+	(segment
+		(start 170.32647 80.725)
+		(end 173.665 80.725)
 		(width 0.2)
 		(layer "F.Cu")
@@
 		(start 170.325735 80.725735)
 		(end 170.32647 80.725)
-		(width 0.2)
-		(layer "F.Cu")
-		(net 6)
-	)
-	(segment
-		(start 170.32647 80.725)
-		(end 173.665 80.725)
-		(width 0.2)
-		(layer "F.Cu")
-		(net 6)
-	)
-	(segment
-		(start 173.665 80.725)
-		(end 174.815 81.875)
-		(width 0.2)
-		(layer "F.Cu")
-		(net 6)
-	)
-	(segment
-		(start 173.53 75.55)
-		(end 173.6 75.62)
 		(width 0.2)
 		(layer "F.Cu")
@@
 			)
 		)
+	)
+	(zone
+		(net 0)
+		(net_name "")
+		(layers "F.Cu" "Edge.Cuts")
+		(hatch edge 0.5)
+		(connect_pads
+			(clearance 0)
+		)
+		(min_thickness 0.25)
+		(filled_areas_thickness no)
+		(keepout
+			(tracks allowed)
+			(vias allowed)
+			(pads allowed)
+			(copperpour not_allowed)
+			(footprints allowed)
+		)
+		(fill
+			(thermal_gap 0.5)
+			(thermal_bridge_width 0.5)
+		)
+		(polygon
+			(pts
+				(xy 173.5 71.5) (xy 174.8 71.5) (xy 174.8 72.7) (xy 173.5 72.7)
+			)
+		)
